File: cweep.kicad_sch (KiCad schematic)
At the start: 73 parts, among them J1 24AWG Hole, J2 24AWG Hole, SW1 SW_Push, SW10 SW_Push, SW11 SW_Push, SW12 SW_Push, SW13 SW_Push, SW14 SW_Push, SW15 SW_Push, SW16 SW_Push, SW17 SW_Push, SW18 SW_SPST, SW19 SW_Omron_B3FS, SW2 SW_Push, SW3 SW_Push, SW4 SW_Push, SW5 SW_Push, SW6 SW_Push, SW7 SW_Push, SW8 SW_Push, SW9 SW_Push, U1 XIAO-nRF52840, U2 BQ25504

Commit message: feat: add solar housing
Parts:
- D1, D10, D11, D12, D13, D14, D15, D16, D17, D2, D3, D4, D5, D6, D7, D8, D9: footprint Diode_SMD:D_SOD-123 -> cweep:D_SOD-123_Reversible
- U2: footprint Package_DFN_QFN:VQFN-16-1EP_3x3mm_P0.5mm_EP1.68x1.68mm -> cweep:VQFN-16-1EP_3x3mm_P0.5mm_EP1.68x1.68mm
Changed lines of the file:
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@@
 			)
 		)
-		(property "Footprint" "Diode_SMD:D_SOD-123"
+		(property "Footprint" "cweep:D_SOD-123_Reversible"
 			(at 114.554 38.354 0)
 			(hide yes)
@@
 			)
 		)
-		(property "Footprint" "Diode_SMD:D_SOD-123"
+		(property "Footprint" "cweep:D_SOD-123_Reversible"
 			(at 127.254 38.354 0)
 			(hide yes)
@@
 			)
 		)
-		(property "Footprint" "Diode_SMD:D_SOD-123"
+		(property "Footprint" "cweep:D_SOD-123_Reversible"
 			(at 127.254 73.914 0)
 			(hide yes)
@@
 			)
 		)
-		(property "Footprint" "Diode_SMD:D_SOD-123"
+		(property "Footprint" "cweep:D_SOD-123_Reversible"
 			(at 152.654 73.914 0)
 			(hide yes)
@@
 			)
 		)
-		(property "Footprint" "Diode_SMD:D_SOD-123"
+		(property "Footprint" "cweep:D_SOD-123_Reversible"
 			(at 127.254 56.134 0)
 			(hide yes)
@@
 			)
 		)
-		(property "Footprint" "Diode_SMD:D_SOD-123"
+		(property "Footprint" "cweep:D_SOD-123_Reversible"
 			(at 114.554 73.914 0)
 			(hide yes)
@@
 			)
 		)
-		(property "Footprint" "Diode_SMD:D_SOD-123"
+		(property "Footprint" "cweep:D_SOD-123_Reversible"
 			(at 152.654 56.134 0)
 			(hide yes)
@@
 			)
 		)
-		(property "Footprint" "Diode_SMD:D_SOD-123"
+		(property "Footprint" "cweep:D_SOD-123_Reversible"
 			(at 139.954 73.914 0)
 			(hide yes)
@@
 			)
 		)
-		(property "Footprint" "Diode_SMD:D_SOD-123"
+		(property "Footprint" "cweep:D_SOD-123_Reversible"
 			(at 139.954 56.134 0)
 			(hide yes)
@@
 			)
 		)
-		(property "Footprint" "Diode_SMD:D_SOD-123"
+		(property "Footprint" "cweep:D_SOD-123_Reversible"
 			(at 101.854 73.914 0)
 			(hide yes)
@@
 			)
 		)
-		(property "Footprint" "Package_DFN_QFN:VQFN-16-1EP_3x3mm_P0.5mm_EP1.68x1.68mm"
+		(property "Footprint" "cweep:VQFN-16-1EP_3x3mm_P0.5mm_EP1.68x1.68mm"
 			(at 50.8 59.69 0)
 			(hide yes)
@@
 			)
 		)
-		(property "Footprint" "Diode_SMD:D_SOD-123"
+		(property "Footprint" "cweep:D_SOD-123_Reversible"
 			(at 101.854 91.694 0)
 			(hide yes)
@@
 			)
 		)
-		(property "Footprint" "Diode_SMD:D_SOD-123"
+		(property "Footprint" "cweep:D_SOD-123_Reversible"
 			(at 152.654 38.354 0)
 			(hide yes)
@@
 			)
 		)
-		(property "Footprint" "Diode_SMD:D_SOD-123"
+		(property "Footprint" "cweep:D_SOD-123_Reversible"
 			(at 114.554 91.694 0)
 			(hide yes)
@@
 			)
 		)
-		(property "Footprint" "Diode_SMD:D_SOD-123"
+		(property "Footprint" "cweep:D_SOD-123_Reversible"
 			(at 139.954 38.354 0)
 			(hide yes)
@@
 			)
 		)
-		(property "Footprint" "Diode_SMD:D_SOD-123"
+		(property "Footprint" "cweep:D_SOD-123_Reversible"
 			(at 114.554 56.134 0)
 			(hide yes)
@@
 			)
 		)
-		(property "Footprint" "Diode_SMD:D_SOD-123"
+		(property "Footprint" "cweep:D_SOD-123_Reversible"
 			(at 101.854 38.354 0)
 			(hide yes)
@@
 			)
 		)
-		(property "Footprint" "Diode_SMD:D_SOD-123"
+		(property "Footprint" "cweep:D_SOD-123_Reversible"
 			(at 101.854 56.134 0)
 			(hide yes)
